File: hardware/STM32F446_memory_demo1/power_supply.kicad_sch (KiCad schematic)
At the start: 0 parts

Commit message: some schematics
Parts:
- added C401, C402, C403, C404: 1uF, Capacitor_SMD:C_0603_1608Metric, symbol Device:C_Small
- added U401: BU33SD5WG-TR, Package_TO_SOT_SMD:SOT-23-5, symbol WITNS_ROHM:BU33SD5WG-TR
- added U402: BU18SD2MG-MTR, Package_TO_SOT_SMD:SOT-23-5, symbol WITNS_ROHM:BU18SD2MG-MTR
Connections:
- new net +1V8: C404.1, U402.5 (OUT)
- new net +3.3V: C402.1, C403.1, U401.5 (OUT), U402.1 (IN), U402.3 (STBY)
- new net GND: C401.2, C402.2, C403.2, C404.2, U401.2 (GND), U402.2 (GND)
- new net VBUS: C401.1, U401.1 (IN), U401.3 (STBY)
