File: hardware/STM32F446_memory_demo1/sdram.kicad_sch (KiCad schematic)
At the start: 1 part, among them U201 IS42S16400J-6TLI

Commit message: some schematics
Parts:
- added C201, C202, C203, C204, C205, C206, C207: 100nF, Capacitor_SMD:C_0603_1608Metric, symbol Device:C_Small
Connections:
- net +3.3V: now also C201.1, C202.1, C203.1, C204.1, C205.1, C206.1, C207.1
- net GND: now also C201.2, C202.2, C203.2, C204.2, C205.2, C206.2, C207.2
