File: hardware/STM32F446_memory_demo1/STM32F446_memory_demo1.kicad_pcb (KiCad board)
At the start: 2 copper layers, 10 parts, among them U201 IS42S16400J-6TLI, U301 STM32F446ZCT6, Y301 16MHz

Commit message: some schematics
Parts:
- added C201: 100nF, Capacitor_SMD:C_0603_1608Metric, F.Cu at (91.0, 108.0)
- added C202: 100nF, Capacitor_SMD:C_0603_1608Metric, F.Cu at (89.0, 108.0)
- added C203: 100nF, Capacitor_SMD:C_0603_1608Metric, F.Cu at (85.0, 109.0)
- added C204: 100nF, Capacitor_SMD:C_0603_1608Metric, F.Cu at (81.0, 109.0)
- added C205: 100nF, Capacitor_SMD:C_0603_1608Metric, F.Cu at (69.0, 108.0)
- added C206: 100nF, Capacitor_SMD:C_0603_1608Metric, F.Cu at (81.0, 125.0)
- added C207: 100nF, Capacitor_SMD:C_0603_1608Metric, F.Cu at (88.0, 125.0)
- added C306: 1uF, Capacitor_SMD:C_0603_1608Metric, F.Cu at (61.0, 97.0)
- added C307: 10nF, Capacitor_SMD:C_0603_1608Metric, F.Cu at (65.0, 97.0)
- added C308: 1uF, Capacitor_SMD:C_0603_1608Metric, F.Cu at (63.0, 97.0)
- added C309: 10nF, Capacitor_SMD:C_0603_1608Metric, F.Cu at (67.0, 97.0)
- added C310: 1uF, Capacitor_SMD:C_0603_1608Metric, F.Cu at (60.0, 80.0)
- added C311: 100nF, Capacitor_SMD:C_0603_1608Metric, F.Cu at (67.0, 86.0)
- added C312: 100nF, Capacitor_SMD:C_0603_1608Metric, F.Cu at (67.0, 93.0)
- added C313: 100nF, Capacitor_SMD:C_0603_1608Metric, F.Cu at (72.0, 100.0)
- added C314: 100nF, Capacitor_SMD:C_0603_1608Metric, F.Cu at (78.5, 100.0)
- added C315: 100nF, Capacitor_SMD:C_0603_1608Metric, F.Cu at (83.5, 100.0)
- added C316: 100nF, Capacitor_SMD:C_0603_1608Metric, F.Cu at (92.0, 99.0)
- added C317: 100nF, Capacitor_SMD:C_0603_1608Metric, F.Cu at (93.0, 90.5)
- added C318: 100nF, Capacitor_SMD:C_0603_1608Metric, F.Cu at (92.0, 75.0)
- added C319: 100nF, Capacitor_SMD:C_0603_1608Metric, F.Cu at (83.0, 74.0)
- added C320: 1uF, Capacitor_SMD:C_0603_1608Metric, F.Cu at (96.0, 85.0)
- added C321: 100nF, Capacitor_SMD:C_0603_1608Metric, F.Cu at (78.0, 74.0)
- added C322: 100nF, Capacitor_SMD:C_0603_1608Metric, F.Cu at (94.0, 85.0)
- added C323: 100nF, Capacitor_SMD:C_0603_1608Metric, F.Cu at (68.0, 75.0)
- added C401: 1uF, Capacitor_SMD:C_0603_1608Metric, F.Cu at (107.0, 71.0)
- added C402: 1uF, Capacitor_SMD:C_0603_1608Metric, F.Cu at (101.0, 71.0)
- added C403: 1uF, Capacitor_SMD:C_0603_1608Metric, F.Cu at (107.0, 66.0)
- added C404: 1uF, Capacitor_SMD:C_0603_1608Metric, F.Cu at (101.0, 66.0)
- added J601: Micro_SD_Card_Det, Connector_Card:microSD_HC_Hirose_DM3AT-SF-PEJM5, F.Cu at (86.0, 62.0)
- added J701: USB_C_Receptacle_USB2.0, Connector_USB:USB_C_Receptacle_HRO_TYPE-C-31-M-12, F.Cu at (111.0, 81.0)
- added L301: 39nH, Inductor_SMD:L_0603_1608Metric, F.Cu at (59.0, 97.0)
- added R701: 5.1k, Resistor_SMD:R_0603_1608Metric_Pad0.98x0.95mm_HandSolder, F.Cu at (104.0, 85.0)
- added R702: 5.1k, Resistor_SMD:R_0603_1608Metric_Pad0.98x0.95mm_HandSolder, F.Cu at (104.0, 76.0)
- added U401: BU33SD5WG-TR, Package_TO_SOT_SMD:SOT-23-5, F.Cu at (104.0, 71.0)
- added U402: BU18SD2MG-MTR, Package_TO_SOT_SMD:SOT-23-5, F.Cu at (104.0, 66.0)
- added U501: SGTL5000XNLA3, Package_DFN_QFN:QFN-20-1EP_3x3mm_P0.4mm_EP1.65x1.65mm, F.Cu at (102.0, 112.0)
- added U701: USBLC6-2SC6, Package_TO_SOT_SMD:SOT-23-6, F.Cu at (102.0, 81.0)
- moved U201 4.12 mm to (80.0, 117.0)
- moved C301 1.03 mm to (61.0, 86.0)
- moved C302 1.00 mm to (61.0, 92.0)
- moved C303 1.00 mm to (65.0, 93.0)
- moved R301 0.50 mm to (74.5, 73.0), turned to 90 degrees
Connections:
- U301 pad 103: unconnected-(U301-Pad103) -> /STM32F446/USB_D-
- U301 pad 104: unconnected-(U301-Pad104) -> /STM32F446/USB_D+
- U301 pad 111: unconnected-(U301-Pad111) -> /SD Card/DAT2
- U301 pad 112: unconnected-(U301-Pad112) -> /SD Card/DAT3
- U301 pad 113: unconnected-(U301-Pad113) -> /SD Card/CLK
- U301 pad 116: unconnected-(U301-Pad116) -> /SD Card/CMD
- U301 pad 32: unconnected-(U301-Pad32) -> +3.3VA
- U301 pad 33: unconnected-(U301-Pad33) -> +3.3VA
- U301 pad 98: unconnected-(U301-Pad98) -> /SD Card/DAT0
- U301 pad 99: unconnected-(U301-Pad99) -> /SD Card/DAT1

Commit message: added a lot of stuff a long time ago :S
Parts:
- added C501: 100nF, Capacitor_SMD:C_0603_1608Metric, F.Cu at (59.0, 68.0)
- added R501: 2.2k, Resistor_SMD:R_0603_1608Metric, F.Cu at (63.0, 65.5)
- added R502: 2.2k, Resistor_SMD:R_0603_1608Metric, F.Cu at (59.0, 65.5)
- added R601: 47k, Resistor_SMD:R_0603_1608Metric, F.Cu at (83.0, 66.5)
- added R602: 47k, Resistor_SMD:R_0603_1608Metric, F.Cu at (85.0, 66.5)
- added R603: 47k, Resistor_SMD:R_0603_1608Metric, F.Cu at (87.0, 66.5)
- added R604: 47k, Resistor_SMD:R_0603_1608Metric, F.Cu at (89.0, 66.5)
- added R605: 47k, Resistor_SMD:R_0603_1608Metric, F.Cu at (91.0, 66.5)
- moved U501 56.9 mm to (60.5, 73.0)
- moved J601 7.00 mm to (86.0, 55.0)
Connections:
- J601 pad 10: unconnected-(J601-Pad10) -> /SD Card/DETECT
- J601 pad 11: unconnected-(J601-Pad11) -> GND
- J601 pad 4: unconnected-(J601-Pad4) -> +3.3V
- J601 pad 6: unconnected-(J601-Pad6) -> GND
- J601 pad 9: unconnected-(J601-Pad9) -> GND
- U301 pad 1: unconnected-(U301-Pad1) -> /Audio CODEC/SYS_MCLK
- U301 pad 139: unconnected-(U301-Pad139) -> /Audio CODEC/CTRL_SCL
- U301 pad 140: unconnected-(U301-Pad140) -> /Audio CODEC/CTRL_SDA
- U301 pad 2: unconnected-(U301-Pad2) -> /Audio CODEC/DOUT
- U301 pad 3: unconnected-(U301-Pad3) -> /Audio CODEC/LRCLK
- U301 pad 4: unconnected-(U301-Pad4) -> /Audio CODEC/SCLK
- U301 pad 5: unconnected-(U301-Pad5) -> /Audio CODEC/DIN
- U301 pad 97: unconnected-(U301-Pad97) -> /SD Card/DETECT
- U501 pad 12: unconnected-(U501-Pad12) -> +3.3V
- U501 pad 13: unconnected-(U501-Pad13) -> /Audio CODEC/SYS_MCLK
- U501 pad 14: unconnected-(U501-Pad14) -> /Audio CODEC/LRCLK
- U501 pad 15: unconnected-(U501-Pad15) -> /Audio CODEC/SCLK
- U501 pad 16: unconnected-(U501-Pad16) -> /Audio CODEC/DOUT
- U501 pad 17: unconnected-(U501-Pad17) -> /Audio CODEC/DIN
- U501 pad 18: unconnected-(U501-Pad18) -> /Audio CODEC/CTRL_SDA
- U501 pad 19: unconnected-(U501-Pad19) -> /Audio CODEC/CTRL_SCL
- U501 pad 20: unconnected-(U501-Pad20) -> +1V8
- U501 pad 3: unconnected-(U501-Pad3) -> +3.3V
- U501 pad 5: unconnected-(U501-Pad5) -> Net-(U501-Pad5)
