File: hardware/STM32F446_memory_demo1/audio_codec.kicad_sch (KiCad schematic)
At the start: 0 parts

Commit message: some schematics
Parts:
- added U501: SGTL5000XNLA3, Package_DFN_QFN:QFN-20-1EP_3x3mm_P0.4mm_EP1.65x1.65mm, symbol Audio:SGTL5000XNLA3
Changed lines of the file:
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@@
 (kicad_sch (version 20211123) (generator eeschema)
   (paper "A4")
+  (symbol (lib_id "Audio:SGTL5000XNLA3") (at 147.32 93.98 0) (unit 1)
+    (in_bom yes) (on_board yes) (fields_autoplaced)
+    (property "Reference" "U501" (id 0) (at 149.3394 122.555 0)
+      (effects (font (size 1.27 1.27)) (justify left))
+    )
+    (property "Value" "SGTL5000XNLA3" (id 1) (at 149.3394 125.095 0)
+      (effects (font (size 1.27 1.27)) (justify left))
+    )
+    (property "Footprint" "Package_DFN_QFN:QFN-20-1EP_3x3mm_P0.4mm_EP1.65x1.65mm" (id 2) (at 147.32 93.98 0)
+      (effects (font (size 1.27 1.27)) hide)
+    )
+    (property "Datasheet" "https://www.nxp.com/docs/en/data-sheet/SGTL5000.pdf" (id 3) (at 147.32 93.98 0)
+      (effects (font (size 1.27 1.27)) hide)
+    )
+    (pin "1")
+    (pin "10")
+    (pin "11")
+    (pin "12")
+    (pin "13")
+    (pin "14")
+    (pin "15")
+    (pin "16")
+    (pin "17")
+    (pin "18")
+    (pin "19")
+    (pin "2")
+    (pin "20")
+    (pin "21")
+    (pin "3")
+    (pin "4")
+    (pin "5")
+    (pin "6")
+    (pin "7")
+    (pin "8")
+    (pin "9")
+  )
 )

Commit message: added a lot of stuff a long time ago :S
Parts:
- added C501: 100nF, Capacitor_SMD:C_0603_1608Metric, symbol Device:C_Small
- added R501, R502: 2.2k, Resistor_SMD:R_0603_1608Metric, symbol Device:R_Small
Connections:
- net +3.3V: now reaches U501.12 (VDDIO)
- net +3.3V: now also U501.3 (VDDA), R501.1, R502.1
- net SYS_MCLK: now reaches U501.13 (SYS_MCLK)
- net LRCLK: now reaches U501.14 (I2S_LRCLK)
- net SCLK: now reaches U501.15 (I2S_SCLK)
- net DOUT: now reaches U501.16 (I2S_DOUT)
- net DIN: now reaches U501.17 (I2S_DIN)
- net CTRL_SDA: now reaches U501.18 (CTRL_DATA)
- net CTRL_SDA: now also R502.2
- net CTRL_SCL: now reaches U501.19 (CTRL_CLK)
- net CTRL_SCL: now also R501.2
- net +1V8: now reaches U501.20 (VDDD)
- net at U501.5 (VAG): now also C501.1
- new net GND: C501.2
Changed lines of the file:
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@@
 (kicad_sch (version 20211123) (generator eeschema)
   (paper "A4")
+  (junction (at 96.52 114.3) (diameter 0) (color 0 0 0 0)
+  )
+  (junction (at 102.87 111.76) (diameter 0) (color 0 0 0 0)
+  )
+  (junction (at 96.52 104.14) (diameter 0) (color 0 0 0 0)
+  )
+  (wire (pts (xy 96.52 104.14) (xy 102.87 104.14))
+    (stroke (width 0) (type default) (color 0 0 0 0))
+  )
+  (wire (pts (xy 132.08 73.66) (xy 100.33 73.66))
+    (stroke (width 0) (type default) (color 0 0 0 0))
+  )
+  (wire (pts (xy 96.52 110.49) (xy 96.52 114.3))
+    (stroke (width 0) (type default) (color 0 0 0 0))
+  )
+  (wire (pts (xy 152.4 63.5) (xy 152.4 66.04))
+    (stroke (width 0) (type default) (color 0 0 0 0))
+  )
+  (wire (pts (xy 100.33 73.66) (xy 100.33 77.47))
+    (stroke (width 0) (type default) (color 0 0 0 0))
+  )
+  (wire (pts (xy 100.33 82.55) (xy 100.33 88.9))
+    (stroke (width 0) (type default) (color 0 0 0 0))
+  )
+  (wire (pts (xy 102.87 104.14) (xy 102.87 105.41))
+    (stroke (width 0) (type default) (color 0 0 0 0))
+  )
+  (wire (pts (xy 92.71 111.76) (xy 102.87 111.76))
+    (stroke (width 0) (type default) (color 0 0 0 0))
+  )
+  (wire (pts (xy 96.52 114.3) (xy 132.08 114.3))
+    (stroke (width 0) (type default) (color 0 0 0 0))
+  )
+  (wire (pts (xy 142.24 63.5) (xy 142.24 66.04))
+    (stroke (width 0) (type default) (color 0 0 0 0))
+  )
+  (wire (pts (xy 147.32 63.5) (xy 147.32 66.04))
+    (stroke (width 0) (type default) (color 0 0 0 0))
+  )
+  (wire (pts (xy 96.52 102.87) (xy 96.52 104.14))
+    (stroke (width 0) (type default) (color 0 0 0 0))
+  )
+  (wire (pts (xy 102.87 110.49) (xy 102.87 111.76))
+    (stroke (width 0) (type default) (color 0 0 0 0))
+  )
+  (wire (pts (xy 92.71 114.3) (xy 96.52 114.3))
+    (stroke (width 0) (type default) (color 0 0 0 0))
+  )
+  (wire (pts (xy 96.52 104.14) (xy 96.52 105.41))
+    (stroke (width 0) (type default) (color 0 0 0 0))
+  )
+  (wire (pts (xy 102.87 111.76) (xy 132.08 111.76))
+    (stroke (width 0) (type default) (color 0 0 0 0))
+  )
+  (hierarchical_label "DOUT" (shape input) (at 132.08 104.14 180)
+    (effects (font (size 1.27 1.27)) (justify right))
+  )
+  (hierarchical_label "CTRL_SDA" (shape input) (at 92.71 111.76 180)
+    (effects (font (size 1.27 1.27)) (justify right))
+  )
+  (hierarchical_label "CTRL_SCL" (shape input) (at 92.71 114.3 180)
+    (effects (font (size 1.27 1.27)) (justify right))
+  )
+  (hierarchical_label "DIN" (shape input) (at 132.08 106.68 180)
+    (effects (font (size 1.27 1.27)) (justify right))
+  )
+  (hierarchical_label "SYS_MCLK" (shape input) (at 132.08 93.98 180)
+    (effects (font (size 1.27 1.27)) (justify right))
+  )
+  (hierarchical_label "SCLK" (shape input) (at 132.08 101.6 180)
+    (effects (font (size 1.27 1.27)) (justify right))
+  )
+  (hierarchical_label "LRCLK" (shape input) (at 132.08 99.06 180)
+    (effects (font (size 1.27 1.27)) (justify right))
+  )
+  (symbol (lib_id "power:+3.3V") (at 96.52 102.87 0) (unit 1)
+    (in_bom yes) (on_board yes) (fields_autoplaced)
+    (property "Reference" "#PWR0133" (id 0) (at 96.52 106.68 0)
+      (effects (font (size 1.27 1.27)) hide)
+    )
+    (property "Value" "+3.3V" (id 1) (at 96.52 97.79 0))
+    (property "Footprint" "" (id 2) (at 96.52 102.87 0)
+      (effects (font (size 1.27 1.27)) hide)
+    )
+    (property "Datasheet" "" (id 3) (at 96.52 102.87 0)
+      (effects (font (size 1.27 1.27)) hide)
+    )
+    (pin "1")
+  )
+  (symbol (lib_id "power:GND") (at 100.33 88.9 0) (unit 1)
+    (in_bom yes) (on_board yes) (fields_autoplaced)
+    (property "Reference" "#PWR0132" (id 0) (at 100.33 95.25 0)
+      (effects (font (size 1.27 1.27)) hide)
+    )
+    (property "Value" "GND" (id 1) (at 100.33 93.98 0))
+    (property "Footprint" "" (id 2) (at 100.33 88.9 0)
+      (effects (font (size 1.27 1.27)) hide)
+    )
+    (property "Datasheet" "" (id 3) (at 100.33 88.9 0)
+      (effects (font (size 1.27 1.27)) hide)
+    )
+    (pin "1")
+  )
+  (symbol (lib_id "Device:R_Small") (at 102.87 107.95 0) (unit 1)
+    (in_bom yes) (on_board yes)
+    (property "Reference" "R502" (id 0) (at 99.06 107.95 90))
+    (property "Value" "2.2k" (id 1) (at 100.965 107.95 90))
+    (property "Footprint" "Resistor_SMD:R_0603_1608Metric" (id 2) (at 102.87 107.95 0)
+      (effects (font (size 1.27 1.27)) hide)
+    )
+    (property "Datasheet" "~" (id 3) (at 102.87 107.95 0)
+      (effects (font (size 1.27 1.27)) hide)
+    )
+    (pin "1")
+    (pin "2")
+  )
+  (symbol (lib_id "Device:C_Small") (at 100.33 80.01 0) (mirror y) (unit 1)
+    (in_bom yes) (on_board yes)
+    (property "Reference" "C501" (id 0) (at 101.6 74.295 90)
+      (effects (font (size 1.27 1.27)) (justify right))
+    )
+    (property "Value" "100nF" (id 1) (at 101.6 81.28 90)
+      (effects (font (size 1.27 1.27)) (justify right))
+    )
+    (property "Footprint" "Capacitor_SMD:C_0603_1608Metric" (id 2) (at 100.33 80.01 0)
+      (effects (font (size 1.27 1.27)) hide)
+    )
+    (property "Datasheet" "~" (id 3) (at 100.33 80.01 0)
+      (effects (font (size 1.27 1.27)) hide)
+    )
+    (pin "1")
+    (pin "2")
+  )
+  (symbol (lib_id "Device:R_Small") (at 96.52 107.95 0) (unit 1)
+    (in_bom yes) (on_board yes)
+    (property "Reference" "R501" (id 0) (at 92.71 107.95 90))
+    (property "Value" "2.2k" (id 1) (at 94.615 107.95 90))
+    (property "Footprint" "Resistor_SMD:R_0603_1608Metric" (id 2) (at 96.52 107.95 0)
+      (effects (font (size 1.27 1.27)) hide)
+    )
+    (property "Datasheet" "~" (id 3) (at 96.52 107.95 0)
+      (effects (font (size 1.27 1.27)) hide)
+    )
+    (pin "1")
+    (pin "2")
+  )
+  (symbol (lib_id "power:+3.3V") (at 142.24 63.5 0) (unit 1)
+    (in_bom yes) (on_board yes) (fields_autoplaced)
+    (property "Reference" "#PWR0130" (id 0) (at 142.24 67.31 0)
+      (effects (font (size 1.27 1.27)) hide)
+    )
+    (property "Value" "+3.3V" (id 1) (at 142.24 58.42 0))
+    (property "Footprint" "" (id 2) (at 142.24 63.5 0)
+      (effects (font (size 1.27 1.27)) hide)
+    )
+    (property "Datasheet" "" (id 3) (at 142.24 63.5 0)
+      (effects (font (size 1.27 1.27)) hide)
+    )
+    (pin "1")
+  )
   (symbol (lib_id "Audio:SGTL5000XNLA3") (at 147.32 93.98 0) (unit 1)
     (in_bom yes) (on_board yes) (fields_autoplaced)
@@
     (pin "9")
   )
+  (symbol (lib_id "power:+3.3V") (at 152.4 63.5 0) (unit 1)
+    (in_bom yes) (on_board yes) (fields_autoplaced)
+    (property "Reference" "#PWR0131" (id 0) (at 152.4 67.31 0)
+      (effects (font (size 1.27 1.27)) hide)
+    )
+    (property "Value" "+3.3V" (id 1) (at 152.4 58.42 0))
+    (property "Footprint" "" (id 2) (at 152.4 63.5 0)
+      (effects (font (size 1.27 1.27)) hide)
+    )
+    (property "Datasheet" "" (id 3) (at 152.4 63.5 0)
+      (effects (font (size 1.27 1.27)) hide)
+    )
+    (pin "1")
+  )
+  (symbol (lib_id "power:+1V8") (at 147.32 63.5 0) (unit 1)
+    (in_bom yes) (on_board yes) (fields_autoplaced)
+    (property "Reference" "#PWR0129" (id 0) (at 147.32 67.31 0)
+      (effects (font (size 1.27 1.27)) hide)
+    )
+    (property "Value" "+1V8" (id 1) (at 147.32 58.42 0))
+    (property "Footprint" "" (id 2) (at 147.32 63.5 0)
+      (effects (font (size 1.27 1.27)) hide)
+    )
+    (property "Datasheet" "" (id 3) (at 147.32 63.5 0)
+      (effects (font (size 1.27 1.27)) hide)
+    )
+    (pin "1")
+  )
 )
