File: hardware/STM32F446_memory_demo1/stm32f446.kicad_sch (KiCad schematic)
At the start: 9 parts, among them U301 STM32F446ZCT6, Y301 16MHz

Commit message: some schematics
Parts:
- added C306, C308, C310, C320: 1uF, Capacitor_SMD:C_0603_1608Metric, symbol Device:C_Small
- added C307, C309: 10nF, Capacitor_SMD:C_0603_1608Metric, symbol Device:C_Small
- added C311, C312, C313, C314, C315, C316, C317, C318, C319, C321, C322, C323: 100nF, Capacitor_SMD:C_0603_1608Metric, symbol Device:C_Small
- added L301: 39nH, Inductor_SMD:L_0603_1608Metric, symbol Device:L_Small
Connections:
- net +3.3V: now also C310.1, C311.1, C312.1, C313.1, C314.1, C315.1, C316.1, C317.1, C318.1, C319.1, C320.1, C321.1, C322.1, C323.1, L301.1
- net GND: now also C306.2, C307.2, C308.2, C309.2, C310.2, C311.2, C312.2, C313.2, C314.2, C315.2, C316.2, C317.2, C318.2, C319.2, C320.2, C321.2, C322.2, C323.2
- net +3.3VA: now reaches U301.32 (VREF+)
- net +3.3VA: now also U301.33 (VDDA), C306.1, C307.1, C308.1, C309.1, L301.2
- net USB_D-: now reaches U301.103 (PA11)
- net USB_D+: now reaches U301.104 (PA12)
- net SDIO_D2: now reaches U301.111 (PC10)
- net SDIO_D3: now reaches U301.112 (PC11)
- net SDIO_CK: now reaches U301.113 (PC12)
- net SDIO_CMD: now reaches U301.116 (PD2)
- net SDIO_D0: now reaches U301.98 (PC8)
- net SDIO_D1: now reaches U301.99 (PC9)

Commit message: added a lot of stuff a long time ago :S
Connections:
- net SAI1_MCLK_A: now reaches U301.1 (PE2)
- net CODEC_I2C_SCL: now reaches U301.139 (PB8)
- net CODEC_I2C_SDA: now reaches U301.140 (PB9)
- net SAI1_SD_B: now reaches U301.2 (PE3)
- net SAI_FS_A: now reaches U301.3 (PE4)
- net SAI1_SCK_A: now reaches U301.4 (PE5)
- net SAI_SD_A: now reaches U301.5 (PE6)
- net SD_DETECT: now reaches U301.97 (PC7)
Other:
- moved on the sheet: C301, C302, C303, C304, C305, C306, C307, C308, C309, C310, C311, C312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
